File: 4_inputs.kicad_sch (KiCad schematic)
At the start: 36 parts, among them K1 G6KU-2, K10 G6KU-2, K11 G6KU-2, K12 G6KU-2, K13 G6KU-2, K14 G6KU-2, K15 G6KU-2, K16 G6KU-2, K2 G6KU-2, K3 G6KU-2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

Commit message: Added bus test points
Other:
- company: (none) -> RPG
- title: (none) -> Relay Block
Changed lines of the file:
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@@
 	(generator_version "10.0")
 	(paper "A3")
+	(title_block
+		(title "Relay Block")
+		(date "2026-06-30")
+		(rev "0.4")
+		(company "RPG")
+	)
 	(junction
 		(at 38.1 72.39)
