File: nbs430_switch.kicad_sch (KiCad schematic)
At the start: 106 parts, among them J1 Conn_01x05_Pin, U1 74ACT125, U10 74HCT595, U11 74HCT595, U12 74ACT125, U13 74HCT595, U14 74ACT125, U15 74HCT595, U16 74ACT125, U17 74HCT595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

Commit message: Added bus test points
Parts:
- added SYM1: Logo_Open_Hardware_Small, Symbol:OSHW-Logo2_14.6x12mm_SilkScreen, symbol Graphic:Logo_Open_Hardware_Small
- added SYM2: Logo_Open_Hardware_Small, Symbol:KiCad-Logo_12mm_SilkScreen, symbol Graphic:Logo_Open_Hardware_Small
- added SYM3: Logo_Open_Hardware_Small, Symbol:WEEE-Logo_8.4x12mm_SilkScreen, symbol Graphic:Logo_Open_Hardware_Small
- added TP1, TP2, TP3, TP4: TestPoint, TestPoint:TestPoint_Loop_D1.80mm_Drill1.0mm_Beaded, symbol Connector:TestPoint
Connections:
- new net bus_A: TP1.1
- new net bus_B: TP2.1
- new net bus_C: TP3.1
- new net bus_D: TP4.1
Other:
- company: reps -> RPG
